File: hardware/bldc_driver/control_elements.sch (KiCad schematic (older format))
At the start: 56 parts, among them J10 U, J11 V, J12 W, J8 Power_Supply, J9 Braking_resistor_terminal, Q1 BSC110N, Q2 BSC110N, Q3 BSC110N, Q4 BSC110N, Q5 BSC110N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

Commit message: Cosmetic - trace improvements
- correcting 3-way trace intersections
Changed lines of the file:
@@
 	-1   0    0    1
 $EndComp
-Text Notes 13050 5850 0    50   ~ 0
+Text Notes 16750 6750 0    50   ~ 0
 https://pl.farnell.com/phoenix-contact/mkds-3-2/terminal-block-wire-to-brd-2pos/dp/2314973?gclid=CjwKCAjw95yJBhAgEiwAmRrutPcA1OBmnMDv9Igh77M6Ev5MJIhGP8Eed6DhvFQ4YEmbCG9QHVjVERoCHNoQAvD_BwE&mckv=s442BoGUX_dc|pcrid|459816541164|plid||kword||match||slid||product|2314973|pgrid|114468574544|ptaid|pla-324939342674|&CMP=KNC-GPL-SHOPPING-Whoop-HI-31-Aug-20&gross_price=true
 Text Label 4550 4600 0    50   ~ 0
